File: nrf24-development-board.kicad_pcb (KiCad board)
At the start: 2 copper layers, 18 parts, among them J1 3.3 Voltage Regulator, J2 Vin, J3 Analog Connectors, J4 FTDI, J5 Digital Connectors, J6 Digital Connectors, J7 Control Connectors, SW1 Reset, U1 ATmega328P-PU, U2 NRF24L01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

Commit message: pcb tracks connected
Parts:
- SW1: footprint Button_Switch_THT:Push_E-Switch_KS01Q01 -> Button_Switch_THT:SW_TH_Tactile_Omron_B3F-10xx
- moved SW1 33.1 mm to (41.8, 52.8), turned to 90 degrees
- moved U2 27.0 mm to (91.5, 77.2), turned to 270 degrees
- moved U1 25.4 mm to (58.5, 45.0)
- moved C2 24.0 mm to (47.0, 86.2)
- moved C3 23.8 mm to (47.0, 91.5)
- moved J2 22.1 mm to (96.8, 31.8)
- moved J1 21.1 mm to (89.0, 37.0)
- moved J4 20.2 mm to (70.5, 31.2)
- moved C1 19.3 mm to (70.5, 36.5)
- moved J5 17.3 mm to (100.2, 70.5)
- moved JP1 16.0 mm to (73.8, 91.5), turned to 270 degrees
- moved J3 15.7 mm to (100.2, 52.0)
- moved J7 15.6 mm to (42.2, 73.2)
- moved C4 14.6 mm to (97.2, 78.2), turned to 0 degrees
- moved J6 13.4 mm to (60.0, 31.3)
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Connections:
- J7 pad 3: GND -> Net-(C1-Pad2)
Routing:
- net +3V3: track 57.7 -> 214.1 mm
- net GND: track 28.9 -> 179.3 mm
- net Net-(J5-Pad2): track 0.00 -> 68.6 mm
- net Net-(J5-Pad3): track 0.00 -> 63.8 mm
- net Net-(J5-Pad6): track 0.00 -> 62.5 mm
- net Net-(J5-Pad4): track 0.00 -> 61.4 mm
- net Net-(C1-Pad2): track 0.00 -> 60.4 mm
- net Net-(J5-Pad1): track 0.00 -> 59.8 mm
- net Net-(J5-Pad5): track 0.00 -> 59.2 mm
- net Net-(J6-Pad8): track 0.00 -> 50.9 mm
- net Net-(J6-Pad7): track 0.00 -> 47.3 mm
- net /Rx: track 0.00 -> 45.9 mm
- net Net-(J6-Pad6): track 0.00 -> 43.7 mm
- net /Aref: track 0.00 -> 40.4 mm
- net Net-(J3-Pad6): track 0.00 -> 36.6 mm
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Other:
- board outline added: 68 x 72 mm

Commit message: Pcb labeled
Parts:
- J1: value 3.3 Voltage Regulator -> 3.3V Regulator
- R1: value R -> 10K
- renumbered U1 to ATMega328
Connections:
- ATMega328 pad 2: /Tx -> /Rx
- J4 pad 3: /Tx -> /Rx
- J6 pad 1: /Tx -> /Rx
Routing:
- net /Tx: track 33.4 -> 0.00 mm
- net /Rx: track 45.9 -> 79.4 mm
- added copper zone on F.Cu, net GND
Other:
- board text added: "+"
- board text added: "-"
- board text added: "104uF"
- board text added: "10K"
- board text added: "10uF"
- board text added: "16 Mhz"
- board text added: "2"
- board text added: "22uF"
- board text added: "3.3 V"
- board text added: "4"
- board text added: "7"
- board text added: "8"
- board text added: "9"
- board text added: "A0"
- board text added: "A1"
- board text added: "A2"
- board text added: "A3"
- board text added: "AREF"
- board text added: "Crystal Jumpers"
- board text added: "GND"
- board text added: "Input Power"
- board text added: "MISO|12"
- board text added: "MOSI|11"
- board text added: "MySensors Development Board Eduardo Marcos V1.0 09/2020"
- board text added: "NRF24L01"
- board text added: "PWM|3"
- board text added: "PWM|5"
- board text added: "PWM|6"
- board text added: "RESET"
- board text added: "RX|0"
- board text added: "Reset"
- board text added: "SCK|13"
- board text added: "SCL|A5"
- board text added: "SDA|A4"
- board text added: "SS|10"
- board text added: "TX|1"
- board text added: "Vi"
- board text added: "Vo"
