File: nrf24-development-board.sch (KiCad schematic (older format))
At the start: 17 parts, among them J1 3.3 Voltage Regulator, J2 Vin, J3 Analog Connectors, J4 FTDI, J5 Digital Connectors, J6 Digital Connectors, J7 Control Connectors, SW1 Reset, U1 ATmega328P-PU, U2 NRF24L01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

Commit message: footprint for schematics
Parts:
- added C4: 10uF, Capacitor_THT:CP_Axial_L10.0mm_D4.5mm_P15.00mm_Horizontal, symbol Device:C
- C1, C2, C3: footprint (none) -> Capacitor_THT:C_Disc_D3.0mm_W1.6mm_P2.50mm
- J1: footprint (none) -> Connector_PinSocket_2.54mm:PinSocket_1x03_P2.54mm_Vertical
- J2: footprint (none) -> Connector_JST:JST_EH_B2B-EH-A_1x02_P2.50mm_Vertical
- J3, J4, J5, J7: footprint (none) -> Connector_PinSocket_2.54mm:PinSocket_1x06_P2.54mm_Vertical
- J6: footprint (none) -> Connector_PinSocket_2.54mm:PinSocket_1x08_P2.54mm_Vertical
- JP1, JP2: footprint (none) -> Connector_PinHeader_2.54mm:PinHeader_1x02_P2.54mm_Vertical
- R1: footprint (none) -> Resistor_THT:R_Axial_DIN0204_L3.6mm_D1.6mm_P7.62mm_Horizontal
- SW1: footprint (none) -> Button_Switch_THT:Push_E-Switch_KS01Q01
- Y1: footprint (none) -> Crystal:Crystal_HC49-4H_Vertical
Connections:
- net +3V3: now also C4.2
- net GND: now also C4.1
- net VDC: no longer names the net of J2.2 (Pin_2)
- net VDC: no longer J1.1 (Pin_1)
Changed lines of the file:
@@
 F 0 "J4" H 4430 6492 50  0000 L CNN
 F 1 "FTDI" H 4430 6401 50  0000 L CNN
-F 2 "" H 4350 6500 50  0001 C CNN
+F 2 "Connector_PinSocket_2.54mm:PinSocket_1x06_P2.54mm_Vertical" H 4350 6500 50  0001 C CNN
 F 3 "~" H 4350 6500 50  0001 C CNN
 	1    4350 6500
@@
 F 0 "J2" H 2568 875 50  0000 C CNN
 F 1 "Vin" H 2568 966 50  0000 C CNN
-F 2 "" H 2650 1200 50  0001 C CNN
+F 2 "Connector_JST:JST_EH_B2B-EH-A_1x02_P2.50mm_Vertical" H 2650 1200 50  0001 C CNN
 F 3 "~" H 2650 1200 50  0001 C CNN
 	1    2650 1200
@@
 F 0 "SW1" H 3250 5685 50  0000 C CNN
 F 1 "Reset" H 3250 5594 50  0000 C CNN
-F 2 "" H 3250 5600 50  0001 C CNN
+F 2 "Button_Switch_THT:Push_E-Switch_KS01Q01" H 3250 5600 50  0001 C CNN
 F 3 "~" H 3250 5600 50  0001 C CNN
 	1    3250 5400
@@
 F 0 "Y1" V 8104 3031 50  0000 L CNN
 F 1 "16Mhz" V 8400 2800 50  0000 L CNN
-F 2 "" H 8150 2900 50  0001 C CNN
+F 2 "Crystal:Crystal_HC49-4H_Vertical" H 8150 2900 50  0001 C CNN
 F 3 "~" H 8150 2900 50  0001 C CNN
 	1    8150 2900
@@
 F 0 "C3" V 8900 3050 50  0000 C CNN
 F 1 "22uF" V 9000 3050 50  0000 C CNN
-F 2 "" H 8788 2900 50  0001 C CNN
+F 2 "Capacitor_THT:C_Disc_D3.0mm_W1.6mm_P2.50mm" H 8788 2900 50  0001 C CNN
 F 3 "~" H 8750 3050 50  0001 C CNN
 	1    8750 3050
@@
 F 0 "C2" V 8498 2750 50  0000 C CNN
 F 1 "22uF" V 8589 2750 50  0000 C CNN
-F 2 "" H 8788 2600 50  0001 C CNN
+F 2 "Capacitor_THT:C_Disc_D3.0mm_W1.6mm_P2.50mm" H 8788 2600 50  0001 C CNN
 F 3 "~" H 8750 2750 50  0001 C CNN
 	1    8750 2750
@@
 F 0 "R1" H 4630 5604 50  0000 R CNN
 F 1 "R" H 4630 5695 50  0000 R CNN
-F 2 "" V 4630 5650 50  0001 C CNN
+F 2 "Resistor_THT:R_Axial_DIN0204_L3.6mm_D1.6mm_P7.62mm_Horizontal" V 4630 5650 50  0001 C CNN
 F 3 "~" H 4700 5650 50  0001 C CNN
 	1    4700 5650
@@
 F 0 "C1" V 4298 6000 50  0000 C CNN
 F 1 "104uF" V 4389 6000 50  0000 C CNN
-F 2 "" H 4588 5850 50  0001 C CNN
+F 2 "Capacitor_THT:C_Disc_D3.0mm_W1.6mm_P2.50mm" H 4588 5850 50  0001 C CNN
 F 3 "~" H 4550 6000 50  0001 C CNN
 	1    4550 6000
@@
 L power:GND #PWR020
 U 1 1 5F53060B
-P 8900 2750
-F 0 "#PWR020" H 8900 2500 50  0001 C CNN
-F 1 "GND" V 8905 2622 50  0000 R CNN
-F 2 "" H 8900 2750 50  0001 C CNN
-F 3 "" H 8900 2750 50  0001 C CNN
-	1    8900 2750
+P 9050 2600
+F 0 "#PWR020" H 9050 2350 50  0001 C CNN
+F 1 "GND" V 9055 2472 50  0000 R CNN
+F 2 "" H 9050 2600 50  0001 C CNN
+F 3 "" H 9050 2600 50  0001 C CNN
+	1    9050 2600
 	0    -1   -1   0
 $EndComp
@@
 F 0 "JP2" H 6950 3114 50  0000 C CNN
 F 1 "Jumper" H 6950 3023 50  0000 C CNN
-F 2 "" H 6950 2850 50  0001 C CNN
+F 2 "Connector_PinHeader_2.54mm:PinHeader_1x02_P2.54mm_Vertical" H 6950 2850 50  0001 C CNN
 F 3 "~" H 6950 2850 50  0001 C CNN
 	1    6950 2850
@@
 F 0 "JP1" H 6500 2850 50  0000 C CNN
 F 1 "Jumper" H 6500 2750 50  0000 C CNN
-F 2 "" H 6500 2950 50  0001 C CNN
+F 2 "Connector_PinHeader_2.54mm:PinHeader_1x02_P2.54mm_Vertical" H 6500 2950 50  0001 C CNN
 F 3 "~" H 6500 2950 50  0001 C CNN
 	1    6500 2950
@@
 F 0 "J1" V 1964 812 50  0000 R CNN
 F 1 "3.3 Voltage Regulator" V 2150 1450 50  0000 R CNN
-F 2 "" H 2000 1000 50  0001 C CNN
+F 2 "Connector_PinSocket_2.54mm:PinSocket_1x03_P2.54mm_Vertical" H 2000 1000 50  0001 C CNN
 F 3 "~" H 2000 1000 50  0001 C CNN
 	1    2000 1000
@@
 	2000 1200 2000 1500
 $Comp
-L power:VDC #PWR07
-U 1 1 5F563114
-P 2850 1100
-F 0 "#PWR07" H 2850 1000 50  0001 C CNN
-F 1 "VDC" H 2865 1273 50  0000 C CNN
-F 2 "" H 2850 1100 50  0001 C CNN
-F 3 "" H 2850 1100 50  0001 C CNN
-	1    2850 1100
-	1    0    0    -1
-$EndComp
-$Comp
-L power:VDC #PWR01
-U 1 1 5F563650
-P 1900 1200
-F 0 "#PWR01" H 1900 1100 50  0001 C CNN
-F 1 "VDC" H 1915 1373 50  0000 C CNN
-F 2 "" H 1900 1200 50  0001 C CNN
-F 3 "" H 1900 1200 50  0001 C CNN
-	1    1900 1200
-	-1   0    0    1
-$EndComp
-$Comp
 L power:+3V3 #PWR010
 U 1 1 5F5870C3
@@
 L power:GND #PWR013
 U 1 1 5F5876B5
-P 4700 1500
-F 0 "#PWR013" H 4700 1250 50  0001 C CNN
-F 1 "GND" H 4705 1327 50  0000 C CNN
-F 2 "" H 4700 1500 50  0001 C CNN
-F 3 "" H 4700 1500 50  0001 C CNN
-	1    4700 1500
+P 4850 1500
+F 0 "#PWR013" H 4850 1250 50  0001 C CNN
+F 1 "GND" H 4855 1327 50  0000 C CNN
+F 2 "" H 4850 1500 50  0001 C CNN
+F 3 "" H 4850 1500 50  0001 C CNN
+	1    4850 1500
 	0    -1   -1   0
 $EndComp
@@
 F 0 "J3" H 3780 3342 50  0000 L CNN
 F 1 "Analog Connectors" H 3780 3251 50  0000 L CNN
-F 2 "" H 3700 3350 50  0001 C CNN
+F 2 "Connector_PinSocket_2.54mm:PinSocket_1x06_P2.54mm_Vertical" H 3700 3350 50  0001 C CNN
 F 3 "~" H 3700 3350 50  0001 C CNN
 	1    3700 3350
@@
 F 0 "J6" H 5830 4242 50  0000 L CNN
 F 1 "Digital Connectors" H 5830 4151 50  0000 L CNN
-F 2 "" H 5750 4250 50  0001 C CNN
+F 2 "Connector_PinSocket_2.54mm:PinSocket_1x08_P2.54mm_Vertical" H 5750 4250 50  0001 C CNN
 F 3 "~" H 5750 4250 50  0001 C CNN
 	1    5750 4250
@@
 F 0 "J5" V 5514 1312 50  0000 R CNN
 F 1 "Digital Connectors" V 5423 1312 50  0000 R CNN
-F 2 "" H 5550 1700 50  0001 C CNN
+F 2 "Connector_PinSocket_2.54mm:PinSocket_1x06_P2.54mm_Vertical" H 5550 1700 50  0001 C CNN
 F 3 "~" H 5550 1700 50  0001 C CNN
 	1    5550 1700
@@
 F 0 "J7" V 7564 1362 50  0000 R CNN
 F 1 "Control Connectors" V 7473 1362 50  0000 R CNN
-F 2 "" H 7600 1750 50  0001 C CNN
+F 2 "Connector_PinSocket_2.54mm:PinSocket_1x06_P2.54mm_Vertical" H 7600 1750 50  0001 C CNN
 F 3 "~" H 7600 1750 50  0001 C CNN
 	1    7600 1750
@@
 	1    0    0    -1
 $EndComp
+$Comp
+L power:PWR_FLAG #FLG0101
+U 1 1 5F68FD00
+P 3150 900
+F 0 "#FLG0101" H 3150 975 50  0001 C CNN
+F 1 "PWR_FLAG" H 3150 1073 50  0000 C CNN
+F 2 "" H 3150 900 50  0001 C CNN
+F 3 "~" H 3150 900 50  0001 C CNN
+	1    3150 900
+	1    0    0    -1
+$EndComp
+Wire Wire Line
+	3150 900  3150 1100
+Wire Wire Line
+	3150 1100 2850 1100
+$Comp
+L power:PWR_FLAG #FLG0102
+U 1 1 5F6934A4
+P 1900 1200
+F 0 "#FLG0102" H 1900 1275 50  0001 C CNN
+F 1 "PWR_FLAG" H 2050 1350 50  0000 C CNN
+F 2 "" H 1900 1200 50  0001 C CNN
+F 3 "~" H 1900 1200 50  0001 C CNN
+	1    1900 1200
+	-1   0    0    1
+$EndComp
+Wire Wire Line
+	8900 2750 8900 2600
+Wire Wire Line
+	8900 2600 9050 2600
+Wire Wire Line
+	4700 1500 4750 1500
+$Comp
+L Device:C C4
+U 1 1 5F6AC024
+P 4500 1000
+F 0 "C4" V 4248 1000 50  0000 C CNN
+F 1 "10uF" V 4339 1000 50  0000 C CNN
+F 2 "Capacitor_THT:CP_Axial_L10.0mm_D4.5mm_P15.00mm_Horizontal" H 4538 850 50  0001 C CNN
+F 3 "~" H 4500 1000 50  0001 C CNN
+	1    4500 1000
+	0    1    1    0
+$EndComp
+Wire Wire Line
+	4350 1000 3500 1000
+Wire Wire Line
+	3500 1000 3500 1500
+Connection ~ 3500 1500
+Wire Wire Line
+	4650 1000 4750 1000
+Wire Wire Line
+	4750 1000 4750 1500
+Connection ~ 4750 1500
+Wire Wire Line
+	4750 1500 4850 1500
 $EndSCHEMATC

Commit message: pcb basic connections
Parts:
- removed C4: 10uF, Capacitor_THT:CP_Axial_L10.0mm_D4.5mm_P15.00mm_Horizontal, symbol Device:C
- added C4: 10uF, Capacitor_THT:CP_Radial_D5.0mm_P2.50mm, symbol Device:CP
Connections:
- net +3V3: now also C4.1
- net GND: now also C4.2
- net VDC: now reaches J2.2 (Pin_2)
- net VDC: now also J1.1 (Pin_1)
Changed lines of the file:
@@
-	1    0    0    -1
-$EndComp
-$Comp
-L power:PWR_FLAG #FLG0101
-U 1 1 5F68FD00
-P 3150 900
-F 0 "#FLG0101" H 3150 975 50  0001 C CNN
-F 1 "PWR_FLAG" H 3150 1073 50  0000 C CNN
-F 2 "" H 3150 900 50  0001 C CNN
-F 3 "~" H 3150 900 50  0001 C CNN
-	1    3150 900
 	1    0    0    -1
 $EndComp
@@
 Wire Wire Line
 	3150 1100 2850 1100
-$Comp
-L power:PWR_FLAG #FLG0102
-U 1 1 5F6934A4
-P 1900 1200
-F 0 "#FLG0102" H 1900 1275 50  0001 C CNN
-F 1 "PWR_FLAG" H 2050 1350 50  0000 C CNN
-F 2 "" H 1900 1200 50  0001 C CNN
-F 3 "~" H 1900 1200 50  0001 C CNN
-	1    1900 1200
-	-1   0    0    1
-$EndComp
 Wire Wire Line
 	8900 2750 8900 2600
@@
 Wire Wire Line
 	4700 1500 4750 1500
-$Comp
-L Device:C C4
-U 1 1 5F6AC024
-P 4500 1000
-F 0 "C4" V 4248 1000 50  0000 C CNN
-F 1 "10uF" V 4339 1000 50  0000 C CNN
-F 2 "Capacitor_THT:CP_Axial_L10.0mm_D4.5mm_P15.00mm_Horizontal" H 4538 850 50  0001 C CNN
-F 3 "~" H 4500 1000 50  0001 C CNN
-	1    4500 1000
-	0    1    1    0
-$EndComp
 Wire Wire Line
 	4350 1000 3500 1000
@@
 Wire Wire Line
 	4750 1500 4850 1500
+$Comp
+L Device:CP C4
+U 1 1 5F6D85D1
+P 4500 1000
+F 0 "C4" V 4755 1000 50  0000 C CNN
+F 1 "10uF" V 4664 1000 50  0000 C CNN
+F 2 "Capacitor_THT:CP_Radial_D5.0mm_P2.50mm" H 4538 850 50  0001 C CNN
+F 3 "~" H 4500 1000 50  0001 C CNN
+	1    4500 1000
+	0    -1   -1   0
+$EndComp
+$Comp
+L power:VDC #PWR?
+U 1 1 5F6E4116
+P 3150 900
+F 0 "#PWR?" H 3150 800 50  0001 C CNN
+F 1 "VDC" H 3165 1073 50  0000 C CNN
+F 2 "" H 3150 900 50  0001 C CNN
+F 3 "" H 3150 900 50  0001 C CNN
+	1    3150 900
+	1    0    0    -1
+$EndComp
+$Comp
+L power:VDC #PWR?
+U 1 1 5F6E480C
+P 1900 1200
+F 0 "#PWR?" H 1900 1100 50  0001 C CNN
+F 1 "VDC" H 1915 1373 50  0000 C CNN
+F 2 "" H 1900 1200 50  0001 C CNN
+F 3 "" H 1900 1200 50  0001 C CNN
+	1    1900 1200
+	-1   0    0    1
+$EndComp
 $EndSCHEMATC

Commit message: Pcb labeled
Parts:
- R1: value R -> 10K
- SW1: footprint Button_Switch_THT:Push_E-Switch_KS01Q01 -> Button_Switch_THT:SW_TH_Tactile_Omron_B3F-10xx
- renumbered U1 to ATMega328
Connections:
- net Tx is gone; now on net Rx: ATMega328.2 (PD0), J4.3 (Pin_3), J6.1 (Pin_1)
- net GND: no longer J7.3 (Pin_3)
- net at ATMega328.1 (~RESET~/PC6), C1.2, R1.1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: now also J7.3 (Pin_3)
Other:
- moved on the sheet: J7
Changed lines of the file:
@@
 $EndDescr
 $Comp
-L MCU_Microchip_ATmega:ATmega328P-PU U1
+L MCU_Microchip_ATmega:ATmega328P-PU ATMega328
 U 1 1 5F4EC4C8
 P 2350 3450
-F 0 "U1" H 1706 3496 50  0000 R CNN
+F 0 "ATMega328" H 1706 3496 50  0000 R CNN
 F 1 "ATmega328P-PU" H 1706 3405 50  0000 R CNN
 F 2 "Package_DIP:DIP-28_W7.62mm" H 2350 3450 50  0001 C CIN
@@
 F 0 "SW1" H 3250 5685 50  0000 C CNN
 F 1 "Reset" H 3250 5594 50  0000 C CNN
-F 2 "Button_Switch_THT:Push_E-Switch_KS01Q01" H 3250 5600 50  0001 C CNN
+F 2 "Button_Switch_THT:SW_TH_Tactile_Omron_B3F-10xx" H 3250 5600 50  0001 C CNN
 F 3 "~" H 3250 5600 50  0001 C CNN
 	1    3250 5400
@@
 P 4700 5650
 F 0 "R1" H 4630 5604 50  0000 R CNN
-F 1 "R" H 4630 5695 50  0000 R CNN
+F 1 "10K" H 4630 5695 50  0000 R CNN
 F 2 "Resistor_THT:R_Axial_DIN0204_L3.6mm_D1.6mm_P7.62mm_Horizontal" V 4630 5650 50  0001 C CNN
 F 3 "~" H 4700 5650 50  0001 C CNN
@@
 P 2350 1950
 F 0 "#PWR04" H 2350 1800 50  0001 C CNN
-F 1 "+3V3" H 2365 2123 50  0000 C CNN
+F 1 "+3V3" H 2250 2050 50  0000 C CNN
 F 2 "" H 2350 1950 50  0001 C CNN
 F 3 "" H 2350 1950 50  0001 C CNN
@@
 P 2450 1950
 F 0 "#PWR06" H 2450 1800 50  0001 C CNN
-F 1 "+3V3" H 2465 2123 50  0000 C CNN
+F 1 "+3V3" H 2550 2050 50  0000 C CNN
 F 2 "" H 2450 1950 50  0001 C CNN
 F 3 "" H 2450 1950 50  0001 C CNN
@@
 	3050 5400 3050 3750
 Connection ~ 3050 3750
-Wire Wire Line
-	3050 3750 4550 3750
 $Comp
 L power:GND #PWR09
@@
 L Connector_Generic:Conn_01x06 J7
 U 1 1 5F657B58
-P 7600 1750
-F 0 "J7" V 7564 1362 50  0000 R CNN
-F 1 "Control Connectors" V 7473 1362 50  0000 R CNN
-F 2 "Connector_PinSocket_2.54mm:PinSocket_1x06_P2.54mm_Vertical" H 7600 1750 50  0001 C CNN
-F 3 "~" H 7600 1750 50  0001 C CNN
-	1    7600 1750
+P 7150 3350
+F 0 "J7" V 7114 2962 50  0000 R CNN
+F 1 "Control Connectors" V 7023 2962 50  0000 R CNN
+F 2 "Connector_PinSocket_2.54mm:PinSocket_1x06_P2.54mm_Vertical" H 7150 3350 50  0001 C CNN
+F 3 "~" H 7150 3350 50  0001 C CNN
+	1    7150 3350
 	0    -1   -1   0
 $EndComp
@@
 L power:GND #PWR015
 U 1 1 5F6596D7
-P 7400 2150
-F 0 "#PWR015" H 7400 1900 50  0001 C CNN
-F 1 "GND" H 7405 1977 50  0000 C CNN
-F 2 "" H 7400 2150 50  0001 C CNN
-F 3 "" H 7400 2150 50  0001 C CNN
-	1    7400 2150
+P 6950 3750
+F 0 "#PWR015" H 6950 3500 50  0001 C CNN
+F 1 "GND" H 6955 3577 50  0000 C CNN
+F 2 "" H 6950 3750 50  0001 C CNN
+F 3 "" H 6950 3750 50  0001 C CNN
+	1    6950 3750
 	1    0    0    -1
 $EndComp
@@
 L power:GND #PWR016
 U 1 1 5F659DA8
-P 7500 1950
-F 0 "#PWR016" H 7500 1700 50  0001 C CNN
-F 1 "GND" H 7505 1777 50  0000 C CNN
-F 2 "" H 7500 1950 50  0001 C CNN
-F 3 "" H 7500 1950 50  0001 C CNN
-	1    7500 1950
-	1    0    0    -1
-$EndComp
-Wire Wire Line
-	7400 2150 7400 1950
+P 7050 3550
+F 0 "#PWR016" H 7050 3300 50  0001 C CNN
+F 1 "GND" H 7055 3377 50  0000 C CNN
+F 2 "" H 7050 3550 50  0001 C CNN
+F 3 "" H 7050 3550 50  0001 C CNN
+	1    7050 3550
+	1    0    0    -1
+$EndComp
+Wire Wire Line
+	6950 3750 6950 3550
 Text Label 1350 2250 0    50   ~ 0
 Aref
 Wire Wire Line
 	1350 2250 1750 2250
-Text Label 7900 1950 3    50   ~ 0
+Text Label 7450 3550 3    50   ~ 0
 Aref
 $Comp
 L power:+3V3 #PWR019
 U 1 1 5F667FC7
-P 7800 2150
-F 0 "#PWR019" H 7800 2000 50  0001 C CNN
-F 1 "+3V3" H 7815 2323 50  0000 C CNN
-F 2 "" H 7800 2150 50  0001 C CNN
-F 3 "" H 7800 2150 50  0001 C CNN
-	1    7800 2150
-	-1   0    0    1
-$EndComp
-Wire Wire Line
-	7600 2150 7600 1950
-Wire Wire Line
-	7800 2150 7800 1950
+P 7350 3750
+F 0 "#PWR019" H 7350 3600 50  0001 C CNN
+F 1 "+3V3" H 7365 3923 50  0000 C CNN
+F 2 "" H 7350 3750 50  0001 C CNN
+F 3 "" H 7350 3750 50  0001 C CNN
+	1    7350 3750
+	-1   0    0    1
+$EndComp
+Wire Wire Line
+	7350 3750 7350 3550
 $Comp
 L power:+3V3 #PWR018
 U 1 1 5F67EC8F
-P 7700 1950
-F 0 "#PWR018" H 7700 1800 50  0001 C CNN
-F 1 "+3V3" H 7715 2123 50  0000 C CNN
-F 2 "" H 7700 1950 50  0001 C CNN
-F 3 "" H 7700 1950 50  0001 C CNN
-	1    7700 1950
-	-1   0    0    1
-$EndComp
-$Comp
-L power:GND #PWR017
-U 1 1 5F67F183
-P 7600 2150
-F 0 "#PWR017" H 7600 1900 50  0001 C CNN
-F 1 "GND" H 7605 1977 50  0000 C CNN
-F 2 "" H 7600 2150 50  0001 C CNN
-F 3 "" H 7600 2150 50  0001 C CNN
-	1    7600 2150
-	1    0    0    -1
+P 7250 3550
+F 0 "#PWR018" H 7250 3400 50  0001 C CNN
+F 1 "+3V3" H 7265 3723 50  0000 C CNN
+F 2 "" H 7250 3550 50  0001 C CNN
+F 3 "" H 7250 3550 50  0001 C CNN
+	1    7250 3550
+	-1   0    0    1
 $EndComp
 Wire Wire Line
@@
 $EndComp
 $Comp
-L power:VDC #PWR?
+L power:VDC #PWR0101
 U 1 1 5F6E4116
 P 3150 900
-F 0 "#PWR?" H 3150 800 50  0001 C CNN
+F 0 "#PWR0101" H 3150 800 50  0001 C CNN
 F 1 "VDC" H 3165 1073 50  0000 C CNN
 F 2 "" H 3150 900 50  0001 C CNN
@@
 $EndComp
 $Comp
-L power:VDC #PWR?
+L power:VDC #PWR0102
 U 1 1 5F6E480C
 P 1900 1200
-F 0 "#PWR?" H 1900 1100 50  0001 C CNN
+F 0 "#PWR0102" H 1900 1100 50  0001 C CNN
 F 1 "VDC" H 1915 1373 50  0000 C CNN
 F 2 "" H 1900 1200 50  0001 C CNN
@@
 	-1   0    0    1
 $EndComp
+Wire Wire Line
+	7150 3750 7150 3550
+Wire Wire Line
+	3050 3750 4550 3750
+Connection ~ 4550 3750
+Wire Wire Line
+	4550 3750 7150 3750
+Text Label 2950 3950 0    50   ~ 0
+Rx
+Text Label 2950 4050 0    50   ~ 0
+Tx
 $EndSCHEMATC
