File: esp32-gateway-board/esp32-gateway-board.kicad_pcb (KiCad board)
At the start: 2 copper layers, 100 x 70 mm, 15 parts, among them J1 Vin, J2 ESP_P1, J3 ESP_P2, J4 LedIn, J5 LedOut, J6 P2_Connectors, J7 P1_Connectors, U1 NRF24L01

Commit message: update readme
Routing:
- added copper zone on F.Cu, net GND
Other:
- board text added: "3V3"
- board text added: "EN"
- board text added: "ESP32 Board"
- board text added: "ESP32 Development Board Eduardo Marcos V1.0 09/2020"
- board text added: "IO01"
- board text added: "IO02"
- board text added: "IO03"
- board text added: "IO04"
- board text added: "IO05"
- board text added: "IO12"
- board text added: "IO13"
- board text added: "IO14"
- board text added: "IO15"
- board text added: "IO16"
- board text added: "IO17"
- board text added: "IO18"
- board text added: "IO19"
- board text added: "IO21"
- board text added: "IO22"
- board text added: "IO23"
- board text added: "IO25"
- board text added: "IO26"
- board text added: "IO27"
- board text added: "IO32"
- board text added: "IO33"
- board text added: "IO34"
- board text added: "IO35"
- board text added: "IO36"
- board text added: "IO39"
- board text added: "VIN"
Changed lines of the file:
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@@
   (general
     (thickness 1.6)
-    (drawings 8)
+    (drawings 40)
     (tracks 94)
     (zones 0)
@@
       (outputformat 1)
       (mirror false)
-      (drillshape 1)
+      (drillshape 0)
       (scaleselection 1)
-      (outputdirectory ""))
+      (outputdirectory "gerber/"))
   )
   (net 0 "")
@@
       (rotate (xyz 0 0 0))
     )
+  )
+  (gr_text "ESP32 Board" (at 50 58) (layer F.SilkS)
+    (effects (font (size 1 1) (thickness 0.15)) (justify right))
+  )
+  (gr_text "ESP32 Development Board\nEduardo Marcos\nV1.0 09/2020" (at 103 49) (layer F.SilkS)
+    (effects (font (size 1 1) (thickness 0.15)) (justify right))
+  )
+  (gr_text IO16 (at 77.5 67.3425) (layer F.SilkS)
+    (effects (font (size 1 1) (thickness 0.15)))
+  )
+  (gr_text IO05 (at 77.5 62.2625) (layer F.SilkS)
+    (effects (font (size 1 1) (thickness 0.15)))
+  )
+  (gr_text IO02 (at 77.5 72.4225) (layer F.SilkS)
+    (effects (font (size 1 1) (thickness 0.15)))
+  )
+  (gr_text GND (at 77.5 77.5025) (layer F.SilkS)
+    (effects (font (size 1 1) (thickness 0.15)))
+  )
+  (gr_text IO21 (at 77.5 54.6425) (layer F.SilkS)
+    (effects (font (size 1 1) (thickness 0.15)))
+  )
+  (gr_text IO18 (at 77.5 59.7225) (layer F.SilkS)
+    (effects (font (size 1 1) (thickness 0.15)))
+  )
+  (gr_text IO15 (at 77.5 74.9625) (layer F.SilkS)
+    (effects (font (size 1 1) (thickness 0.15)))
+  )
+  (gr_text IO17 (at 77.5 64.8025) (layer F.SilkS)
+    (effects (font (size 1 1) (thickness 0.15)))
+  )
+  (gr_text 3V3 (at 77.5 80.0425) (layer F.SilkS)
+    (effects (font (size 1 1) (thickness 0.15)))
+  )
+  (gr_text IO23 (at 77.5 44.4825) (layer F.SilkS)
+    (effects (font (size 1 1) (thickness 0.15)))
+  )
+  (gr_text IO01 (at 77.5 49.5625) (layer F.SilkS)
+    (effects (font (size 1 1) (thickness 0.15)))
+  )
+  (gr_text IO03 (at 77.5 52.1025) (layer F.SilkS)
+    (effects (font (size 1 1) (thickness 0.15)))
+  )
+  (gr_text IO04 (at 77.5 69.8825) (layer F.SilkS)
+    (effects (font (size 1 1) (thickness 0.15)))
+  )
+  (gr_text IO22 (at 77.5 47.0225) (layer F.SilkS)
+    (effects (font (size 1 1) (thickness 0.15)))
+  )
+  (gr_text IO19 (at 77.5 57.1825) (layer F.SilkS)
+    (effects (font (size 1 1) (thickness 0.15)))
+  )
+  (gr_text VIN (at 22.5 79.7925) (layer F.SilkS)
+    (effects (font (size 1 1) (thickness 0.15)))
+  )
+  (gr_text GND (at 22.5 77.2525) (layer F.SilkS)
+    (effects (font (size 1 1) (thickness 0.15)))
+  )
+  (gr_text IO13 (at 22.5 74.7125) (layer F.SilkS)
+    (effects (font (size 1 1) (thickness 0.15)))
+  )
+  (gr_text IO12 (at 22.5 72.1725) (layer F.SilkS)
+    (effects (font (size 1 1) (thickness 0.15)))
+  )
+  (gr_text IO14 (at 22.5 69.6325) (layer F.SilkS)
+    (effects (font (size 1 1) (thickness 0.15)))
+  )
+  (gr_text IO27 (at 22.5 67.0925) (layer F.SilkS)
+    (effects (font (size 1 1) (thickness 0.15)))
+  )
+  (gr_text IO26 (at 22.5 64.5525) (layer F.SilkS)
+    (effects (font (size 1 1) (thickness 0.15)))
+  )
+  (gr_text IO25 (at 22.5 62.0125) (layer F.SilkS)
+    (effects (font (size 1 1) (thickness 0.15)))
+  )
+  (gr_text IO33 (at 22.5 59.4725) (layer F.SilkS)
+    (effects (font (size 1 1) (thickness 0.15)))
+  )
+  (gr_text IO32 (at 22.5 56.9325) (layer F.SilkS)
+    (effects (font (size 1 1) (thickness 0.15)))
+  )
+  (gr_text IO35 (at 22.5 54.3925) (layer F.SilkS)
+    (effects (font (size 1 1) (thickness 0.15)))
+  )
+  (gr_text IO34 (at 22.5 51.8525) (layer F.SilkS)
+    (effects (font (size 1 1) (thickness 0.15)))
+  )
+  (gr_text IO39 (at 22.5 49.3125) (layer F.SilkS)
+    (effects (font (size 1 1) (thickness 0.15)))
+  )
+  (gr_text IO36 (at 22.5 46.7725) (layer F.SilkS)
+    (effects (font (size 1 1) (thickness 0.15)))
+  )
+  (gr_text EN (at 22.5 44.2325) (layer F.SilkS)
+    (effects (font (size 1 1) (thickness 0.15)))
   )
   (gr_line (start 109 23) (end 109 93) (layer Edge.Cuts) (width 0.1))
@@
   (segment (start 97.6 30.6) (end 98.7 31.7) (width 0.25) (layer F.Cu) (net 38))
   (segment (start 92.4 30.6) (end 97.6 30.6) (width 0.25) (layer F.Cu) (net 38))
+  (zone (net 8) (net_name GND) (layer F.Cu) (hatch edge 0.508)
+    (connect_pads (clearance 0.508))
+    (min_thickness 0.254)
+    (fill yes (arc_segments 32) (thermal_gap 0.508) (thermal_bridge_width 0.508))
+    (polygon
+      (pts
+        (xy 109 93) (xy 9 93) (xy 9 23) (xy 109 23)
+      )
+    )
+  )
 )
